Commit message: feat: omniseer display launch working

File: ros_ws/src/omniseer_description/urdf/xacro/omniseer.urdf.xacro (robot description, xacro)
@@ -1,8 +1,7 @@
 <?xml version='1.0' encoding='utf-8'?>
 <robot xmlns:xacro="http://www.ros.org/wiki/xacro" name="omniseer">
-<robot name="omniseer_urdf_export">
     <link name="fl_wheel">
         <inertial>
-            <origin xyz="1.7993153278439422e-09 2s.26380317489938e-09 0.02100000076677828" rpy="0.0 -0.0 0.0" />
+            <origin xyz="1.7993153278439422e-09 2.26380317489938e-09 0.02100000076677828" rpy="0.0 -0.0 0.0" />
             <mass value="0.1449437592188408" />
             <inertia ixx="0.00010654272201079539" iyy="0.00010654272201080037" izz="0.00017047197881125639" ixy="-4.7460314825842516e-20" iyz="-5.1880768019325896e-20" ixz="0.0" />
@@ -11,5 +10,5 @@
             <origin xyz="1.7993155232431945e-09 1.1387656346129211e-09 0.021000000766778337" rpy="1.5707963267948968 1.2281842209915656e-15 3.1554436208840444e-30" />
             <geometry>
-                <mesh filename="meshes/fl_wheel.stl" scale="0.001 0.001 0.001" />
+                <mesh filename="package://omniseer_description/meshes/fl_wheel.stl" scale="0.001 0.001 0.001" />
             </geometry>
         </visual>
@@ -17,5 +16,5 @@
             <origin xyz="1.7993155232431945e-09 1.1387656346129211e-09 0.021000000766778337" rpy="1.5707963267948968 1.2281842209915656e-15 3.1554436208840444e-30" />
             <geometry>
-                <mesh filename="meshes/fl_wheel.stl" scale="0.001 0.001 0.001" />
+                <mesh filename="package://omniseer_description/meshes/fl_wheel.stl" scale="0.001 0.001 0.001" />
             </geometry>
         </collision>
@@ -30,5 +29,5 @@
             <origin xyz="-1.7993151324446899e-09 1.1387656346129211e-09 0.021000000766778337" rpy="1.5707963267948968 1.2281842209915656e-15 3.1554436208840444e-30" />
             <geometry>
-                <mesh filename="meshes/bl_wheel.stl" scale="0.001 0.001 0.001" />
+                <mesh filename="package://omniseer_description/meshes/bl_wheel.stl" scale="0.001 0.001 0.001" />
             </geometry>
         </visual>
@@ -36,5 +35,5 @@
             <origin xyz="-1.7993151324446899e-09 1.1387656346129211e-09 0.021000000766778337" rpy="1.5707963267948968 1.2281842209915656e-15 3.1554436208840444e-30" />
             <geometry>
-                <mesh filename="meshes/bl_wheel.stl" scale="0.001 0.001 0.001" />
+                <mesh filename="package://omniseer_description/meshes/bl_wheel.stl" scale="0.001 0.001 0.001" />
             </geometry>
         </collision>
@@ -49,5 +48,5 @@
             <origin xyz="1.7993155765338997e-09 -1.1387656346129211e-09 0.02100000076677823" rpy="-1.5707963267948966 -1.2281842209915656e-15 -3.1554436208840444e-30" />
             <geometry>
-                <mesh filename="meshes/fr_wheel.stl" scale="0.001 0.001 0.001" />
+                <mesh filename="package://omniseer_description/meshes/fr_wheel.stl" scale="0.001 0.001 0.001" />
             </geometry>
         </visual>
@@ -55,5 +54,5 @@
             <origin xyz="1.7993155765338997e-09 -1.1387656346129211e-09 0.02100000076677823" rpy="-1.5707963267948966 -1.2281842209915656e-15 -3.1554436208840444e-30" />
             <geometry>
-                <mesh filename="meshes/fr_wheel.stl" scale="0.001 0.001 0.001" />
+                <mesh filename="package://omniseer_description/meshes/fr_wheel.stl" scale="0.001 0.001 0.001" />
             </geometry>
         </collision>
@@ -68,5 +67,5 @@
             <origin xyz="-1.7993150791539846e-09 -1.1387656346129211e-09 0.02100000076677823" rpy="-1.5707963267948966 -1.2281842209915656e-15 -3.1554436208840444e-30" />
             <geometry>
-                <mesh filename="meshes/br_wheel.stl" scale="0.001 0.001 0.001" />
+                <mesh filename="package://omniseer_description/meshes/br_wheel.stl" scale="0.001 0.001 0.001" />
             </geometry>
         </visual>
@@ -74,5 +73,5 @@
             <origin xyz="-1.7993150791539846e-09 -1.1387656346129211e-09 0.02100000076677823" rpy="-1.5707963267948966 -1.2281842209915656e-15 -3.1554436208840444e-30" />
             <geometry>
-                <mesh filename="meshes/br_wheel.stl" scale="0.001 0.001 0.001" />
+                <mesh filename="package://omniseer_description/meshes/br_wheel.stl" scale="0.001 0.001 0.001" />
             </geometry>
         </collision>
@@ -87,5 +86,5 @@
             <origin xyz="0.0 0.0 0.0" rpy="0.0 0.0 0.0" />
             <geometry>
-                <mesh filename="meshes/chassis.stl" scale="0.001 0.001 0.001" />
+                <mesh filename="package://omniseer_description/meshes/chassis.stl" scale="0.001 0.001 0.001" />
             </geometry>
         </visual>
@@ -93,5 +92,5 @@
             <origin xyz="0.0 0.0 0.0" rpy="0.0 0.0 0.0" />
             <geometry>
-                <mesh filename="meshes/chassis.stl" scale="0.001 0.001 0.001" />
+                <mesh filename="package://omniseer_description/meshes/chassis.stl" scale="0.001 0.001 0.001" />
             </geometry>
         </collision>
@@ -106,5 +105,5 @@
             <origin xyz="0.0 0.0 -0.15209671" rpy="0.0 -0.0 0.0" />
             <geometry>
-                <mesh filename="meshes/lidar_top.stl" scale="0.001 0.001 0.001" />
+                <mesh filename="package://omniseer_description/meshes/lidar_top.stl" scale="0.001 0.001 0.001" />
             </geometry>
         </visual>
@@ -112,5 +111,5 @@
             <origin xyz="0.0 0.0 -0.15209671" rpy="0.0 -0.0 0.0" />
             <geometry>
-                <mesh filename="meshes/lidar_top.stl" scale="0.001 0.001 0.001" />
+                <mesh filename="package://omniseer_description/meshes/lidar_top.stl" scale="0.001 0.001 0.001" />
             </geometry>
         </collision>
@@ -146,3 +145,9 @@
         <axis xyz="0.0 0.0 1.0" />
     </joint>
+    <link name="base_link"/>
+    <joint name="base_to_chassis" type="fixed">
+    <parent link="base_link"/>
+    <child  link="chassis"/>
+    <origin xyz="0 0 0" rpy="0 0 0"/>
+    </joint>
 </robot>

Commit message: feat: teleoperation script added

File: ros_ws/src/omniseer_description/urdf/xacro/omniseer.urdf.xacro (robot description, xacro)
@@ -1,4 +1,28 @@
 <?xml version='1.0' encoding='utf-8'?>
 <robot xmlns:xacro="http://www.ros.org/wiki/xacro" name="omniseer">
+    <xacro:property name="lx" value="0.0976"/>
+    <xacro:property name="ly" value="0.0866"/>
+    <xacro:property name="wheel_radius" value="0.021"/>
+    <xacro:property name="wheel_joints"
+                    value="['chassis_fl_wheel_joint',
+                            'chassis_fr_wheel_joint',
+                            'chassis_bl_wheel_joint',
+                            'chassis_br_wheel_joint']"/>
+    <xacro:macro name="wheel_transmission" params="joint">
+        <transmission name="${joint}_tr">
+            <type>transmission_interface/SimpleTransmission</type>
+            <joint name="${joint}">
+                <hardwareInterface>hardware_interface/VelocityJointInterface</hardwareInterface>
+            </joint>
+            <actuator name="${joint}_motor">
+                <hardwareInterface>hardware_interface/VelocityJointInterface</hardwareInterface>
+                <mechanicalReduction>1</mechanicalReduction>
+            </actuator>
+        </transmission>
+    </xacro:macro>
+    <xacro:wheel_transmission joint="chassis_fl_wheel_joint"/>
+    <xacro:wheel_transmission joint="chassis_fr_wheel_joint"/>
+    <xacro:wheel_transmission joint="chassis_bl_wheel_joint"/>
+    <xacro:wheel_transmission joint="chassis_br_wheel_joint"/>
     <link name="fl_wheel">
         <inertial>
@@ -147,7 +171,33 @@
     <link name="base_link"/>
     <joint name="base_to_chassis" type="fixed">
-    <parent link="base_link"/>
-    <child  link="chassis"/>
-    <origin xyz="0 0 0" rpy="0 0 0"/>
-    </joint>
+        <parent link="base_link"/>
+        <child  link="chassis"/>
+        <origin xyz="0 0 0" rpy="0 0 0"/>
+    </joint>
+    <ros2_control name="mecanum_hw" type="system">
+        <hardware>
+            <plugin>gazebo_ros2_control/GazeboSystem</plugin>
+        </hardware>
+        <joint name="chassis_fl_wheel_joint">
+            <command_interface name="velocity"/>
+            <state_interface   name="velocity"/>
+        </joint>
+        <joint name="chassis_fr_wheel_joint">
+            <command_interface name="velocity"/>
+            <state_interface   name="velocity"/>
+        </joint>
+        <joint name="chassis_bl_wheel_joint">
+            <command_interface name="velocity"/>
+            <state_interface   name="velocity"/>
+        </joint>
+        <joint name="chassis_br_wheel_joint">
+            <command_interface name="velocity"/>
+            <state_interface   name="velocity"/>
+        </joint>
+    </ros2_control>
+    <gazebo>
+        <plugin name="ros2_control" filename="libgz_ros2_control.so">
+            <update_rate>100</update_rate>
+        </plugin>
+    </gazebo>
 </robot>

Commit message: feat: launch configuration working for simulation

File: ros_ws/src/omniseer_description/urdf/xacro/omniseer.urdf.xacro (robot description, xacro)
@@ -1,7 +1,8 @@
 <?xml version='1.0' encoding='utf-8'?>
 <robot xmlns:xacro="http://www.ros.org/wiki/xacro" name="omniseer">
-    <xacro:property name="lx" value="0.0976"/>
+    <xacro:property name="body_rgba" value="0.0 0.6 1.0 1.0"/>  <!-- cyan-ish -->
+    <xacro:property name="lx" value="0.0974"/>
     <xacro:property name="ly" value="0.0866"/>
-    <xacro:property name="wheel_radius" value="0.021"/>
+    <xacro:property name="wheel_radius" value="0.0485"/>
     <xacro:property name="wheel_joints"
                     value="['chassis_fl_wheel_joint',
@@ -175,28 +176,44 @@
         <origin xyz="0 0 0" rpy="0 0 0"/>
     </joint>
-    <ros2_control name="mecanum_hw" type="system">
+    <ros2_control name="GazeboSimSystem" type="system">
         <hardware>
-            <plugin>gazebo_ros2_control/GazeboSystem</plugin>
+            <plugin>gz_ros2_control/GazeboSimSystem</plugin>
         </hardware>
         <joint name="chassis_fl_wheel_joint">
-            <command_interface name="velocity"/>
+            <command_interface name="velocity">
+                <param name="min">-1</param>
+                <param name="max">1</param>
+            </command_interface>
             <state_interface   name="velocity"/>
         </joint>
         <joint name="chassis_fr_wheel_joint">
-            <command_interface name="velocity"/>
+            <command_interface name="velocity">
+                <param name="min">-1</param>
+                <param name="max">1</param>
+            </command_interface>
             <state_interface   name="velocity"/>
         </joint>
         <joint name="chassis_bl_wheel_joint">
-            <command_interface name="velocity"/>
+            <command_interface name="velocity">
+                <param name="min">-1</param>
+                <param name="max">1</param>
+            </command_interface>
             <state_interface   name="velocity"/>
         </joint>
         <joint name="chassis_br_wheel_joint">
-            <command_interface name="velocity"/>
+            <command_interface name="velocity">
+                <param name="min">-1</param>
+                <param name="max">1</param>
+            </command_interface>
             <state_interface   name="velocity"/>
         </joint>
     </ros2_control>
     <gazebo>
-        <plugin name="ros2_control" filename="libgz_ros2_control.so">
-            <update_rate>100</update_rate>
+        <plugin name="gz_ros2_control::GazeboSimROS2ControlPlugin" filename="libgz_ros2_control-system">
+            <verbose>true</verbose>
+            <parameters>
+                $(find bringup)/config/controllers.yaml
+            </parameters>
+            <controller_manager_prefix_node_name>controller_manager</controller_manager_prefix_node_name>
         </plugin>
     </gazebo>

Commit message: feat: rviz odometry viewer on sim launch

File: ros_ws/src/omniseer_description/urdf/xacro/omniseer.urdf.xacro (robot description, xacro)
@@ -1,5 +1,6 @@
 <?xml version='1.0' encoding='utf-8'?>
-<robot xmlns:xacro="http://www.ros.org/wiki/xacro" name="omniseer">
-    <xacro:property name="body_rgba" value="0.0 0.6 1.0 1.0"/>  <!-- cyan-ish -->
+<robot xmlns:xacro="http://www.ros.org/wiki/xacro" name="omniseer" xmlns:gz="http://gazebosim.org/schema">
+    <xacro:property name="body_rgba"   value="0.671 0.663 0.506 1.0"/>
+    <xacro:property name="sensor_rgba" value="0.0 0.0 0.0 1.0"/>
     <xacro:property name="lx" value="0.0974"/>
     <xacro:property name="ly" value="0.0866"/>
@@ -37,4 +38,7 @@
                 <mesh filename="package://omniseer_description/meshes/fl_wheel.stl" scale="0.001 0.001 0.001" />
             </geometry>
+            <material name='body_mat'>
+                <color rgba="${body_rgba}"/>
+            </material>
         </visual>
         <collision name="fl_wheel_collision">
@@ -56,4 +60,7 @@
                 <mesh filename="package://omniseer_description/meshes/bl_wheel.stl" scale="0.001 0.001 0.001" />
             </geometry>
+            <material name='body_mat'>
+                <color rgba="${body_rgba}"/>
+            </material>
         </visual>
         <collision name="bl_wheel_collision">
@@ -75,4 +82,7 @@
                 <mesh filename="package://omniseer_description/meshes/fr_wheel.stl" scale="0.001 0.001 0.001" />
             </geometry>
+            <material name='body_mat'>
+                <color rgba="${body_rgba}"/>
+            </material>
         </visual>
         <collision name="fr_wheel_collision">
@@ -94,4 +104,7 @@
                 <mesh filename="package://omniseer_description/meshes/br_wheel.stl" scale="0.001 0.001 0.001" />
             </geometry>
+            <material name='body_mat'>
+                <color rgba="${body_rgba}"/>
+            </material>
         </visual>
         <collision name="br_wheel_collision">
@@ -113,4 +126,7 @@
                 <mesh filename="package://omniseer_description/meshes/chassis.stl" scale="0.001 0.001 0.001" />
             </geometry>
+            <material name='body_mat'>
+                <color rgba="${body_rgba}"/>
+            </material>
         </visual>
         <collision name="chassis_collision">
@@ -132,4 +148,7 @@
                 <mesh filename="package://omniseer_description/meshes/lidar_top.stl" scale="0.001 0.001 0.001" />
             </geometry>
+            <material name='sensor_mat'>
+                <color rgba="${sensor_rgba}"/>
+            </material>
         </visual>
         <collision name="lidar_top_collision">
@@ -144,5 +163,5 @@
         <parent link="chassis" />
         <child link="br_wheel" />
-        <axis xyz="0.0 0.0 1.0" />
+        <axis xyz="0.0 0.0 -1.0" />
     </joint>
     <joint name="chassis_fr_wheel_joint" type="continuous">
@@ -150,5 +169,5 @@
         <parent link="chassis" />
         <child link="fr_wheel" />
-        <axis xyz="-0.0 -0.0 1.0" />
+        <axis xyz="-0.0 -0.0 -1.0" />
     </joint>
     <joint name="chassis_bl_wheel_joint" type="continuous">
@@ -164,9 +183,9 @@
         <axis xyz="0.0 0.0 1.0" />
     </joint>
-    <joint name="chassis_lidar_joint" type="continuous">
+    <joint name="chassis_lidar_joint" type="fixed">
         <origin xyz="0.0 0.0 0.15209671" rpy="0.0 -0.0 0.0" />
         <parent link="chassis" />
         <child link="lidar_top" />
-        <axis xyz="0.0 0.0 1.0" />
+        <!-- <axis xyz="0.0 0.0 1.0" /> -->
     </joint>
     <link name="base_link"/>
@@ -186,4 +205,6 @@
             </command_interface>
             <state_interface   name="velocity"/>
+            <state_interface   name="position"/>
+            <state_interface   name="effort"/>
         </joint>
         <joint name="chassis_fr_wheel_joint">
@@ -193,4 +214,6 @@
             </command_interface>
             <state_interface   name="velocity"/>
+            <state_interface   name="position"/>
+            <state_interface   name="effort"/>
         </joint>
         <joint name="chassis_bl_wheel_joint">
@@ -200,4 +223,6 @@
             </command_interface>
             <state_interface   name="velocity"/>
+            <state_interface   name="position"/>
+            <state_interface   name="effort"/>
         </joint>
         <joint name="chassis_br_wheel_joint">
@@ -207,6 +232,60 @@
             </command_interface>
             <state_interface   name="velocity"/>
+            <state_interface   name="position"/>
+            <state_interface   name="effort"/>
         </joint>
     </ros2_control>
+    <gazebo reference='fl_wheel'>
+        <collision>
+            <surface>
+                <friction>
+                    <ode>
+                        <mu>1.0</mu>
+                        <mu2>0.0</mu2>
+                        <fdir1 gz:expressed_in="base_link">1 -1 0</fdir1>
+                    </ode>
+                </friction>
+            </surface>
+        </collision>
+    </gazebo>
+    <gazebo reference='fr_wheel'>
+        <collision>
+            <surface>
+                <friction>
+                <ode>
+                    <mu>1.0</mu>
+                    <mu2>0.0</mu2>
+                    <fdir1 gz:expressed_in="base_link">1 1 0</fdir1>
+                </ode>
+                </friction>
+            </surface>
+        </collision>
+    </gazebo>
+    <gazebo reference='bl_wheel'>
+        <collision>
+            <surface>
+                <friction>
+                    <ode>
+                        <mu>1.0</mu>
+                        <mu2>0.0</mu2>
+                        <fdir1 gz:expressed_in="base_link">1 1 0</fdir1>
+                    </ode>
+                </friction>
+            </surface>
+        </collision>
+    </gazebo>
+    <gazebo reference='br_wheel'>
+        <collision>
+            <surface>
+                <friction>
+                    <ode>
+                        <mu>1.0</mu>
+                        <mu2>0.0</mu2>
+                        <fdir1 gz:expressed_in="base_link">1 -1 0</fdir1>
+                    </ode>
+                </friction>
+            </surface>
+        </collision>
+    </gazebo>
     <gazebo>
         <plugin name="gz_ros2_control::GazeboSimROS2ControlPlugin" filename="libgz_ros2_control-system">

Commit message: feats: analysis package brought in, gz odometry publishing on /model_odom, working on path recorder custom node

File: ros_ws/src/omniseer_description/urdf/xacro/omniseer.urdf.xacro (robot description, xacro)
@@ -1,4 +1,8 @@
 <?xml version='1.0' encoding='utf-8'?>
 <robot xmlns:xacro="http://www.ros.org/wiki/xacro" name="omniseer" xmlns:gz="http://gazebosim.org/schema">
+    <xacro:property name="kp"   value="1e5"/>
+    <xacro:property name="kd"   value="1.0"/>
+    <xacro:property name="mu"   value="1.0"/>
+    <xacro:property name="mu2"   value="0.05"/>
     <xacro:property name="body_rgba"   value="0.671 0.663 0.506 1.0"/>
     <xacro:property name="sensor_rgba" value="0.0 0.0 0.0 1.0"/>
@@ -6,9 +10,4 @@
     <xacro:property name="ly" value="0.0866"/>
     <xacro:property name="wheel_radius" value="0.0485"/>
-    <xacro:property name="wheel_joints"
-                    value="['chassis_fl_wheel_joint',
-                            'chassis_fr_wheel_joint',
-                            'chassis_bl_wheel_joint',
-                            'chassis_br_wheel_joint']"/>
     <xacro:macro name="wheel_transmission" params="joint">
         <transmission name="${joint}_tr">
@@ -187,5 +186,4 @@
         <parent link="chassis" />
         <child link="lidar_top" />
-        <!-- <axis xyz="0.0 0.0 1.0" /> -->
     </joint>
     <link name="base_link"/>
@@ -241,9 +239,15 @@
                 <friction>
                     <ode>
-                        <mu>1.0</mu>
-                        <mu2>0.0</mu2>
+                        <mu>${mu}</mu>
+                        <mu2>${mu2}</mu2>
                         <fdir1 gz:expressed_in="base_link">1 -1 0</fdir1>
                     </ode>
                 </friction>
+                <contact>
+                    <ode>
+                        <kp>${kp}</kp>
+                        <kd>${kd}</kd>
+                    </ode>
+                </contact>
             </surface>
         </collision>
@@ -254,9 +258,15 @@
                 <friction>
                 <ode>
-                    <mu>1.0</mu>
-                    <mu2>0.0</mu2>
+                    <mu>${mu}</mu>
+                    <mu2>${mu2}</mu2>
                     <fdir1 gz:expressed_in="base_link">1 1 0</fdir1>
                 </ode>
                 </friction>
+                <contact>
+                    <ode>
+                        <kp>${kp}</kp>
+                        <kd>${kd}</kd>
+                    </ode>
+                </contact>
             </surface>
         </collision>
@@ -267,9 +277,15 @@
                 <friction>
                     <ode>
-                        <mu>1.0</mu>
-                        <mu2>0.0</mu2>
+                        <mu>${mu}</mu>
+                        <mu2>${mu2}</mu2>
                         <fdir1 gz:expressed_in="base_link">1 1 0</fdir1>
                     </ode>
                 </friction>
+                <contact>
+                    <ode>
+                        <kp>${kp}</kp>
+                        <kd>${kd}</kd>
+                    </ode>
+                </contact>
             </surface>
         </collision>
@@ -280,9 +296,15 @@
                 <friction>
                     <ode>
-                        <mu>1.0</mu>
-                        <mu2>0.0</mu2>
+                        <mu>${mu}</mu>
+                        <mu2>${mu2}</mu2>
                         <fdir1 gz:expressed_in="base_link">1 -1 0</fdir1>
                     </ode>
                 </friction>
+                <contact>
+                    <ode>
+                        <kp>${kp}</kp>
+                        <kd>${kd}</kd>
+                    </ode>
+                </contact>
             </surface>
         </collision>
@@ -297,3 +319,12 @@
         </plugin>
     </gazebo>
+    <gazebo>
+        <plugin filename="gz-sim-odometry-publisher-system" name="gz::sim::systems::OdometryPublisher">
+            <dimensions>3</dimensions>
+            <odom_publish_frequency>50</odom_publish_frequency>
+            <odom_frame>odom</odom_frame>
+            <odom_topic>/model_odom</odom_topic>
+            <robot_base_frame>base_link</robot_base_frame>
+        </plugin>
+    </gazebo>
 </robot>
