Commit message: feat: holonomic motion working in gz

File: ros_ws/src/omniseer_description/urdf/xacro/omniseer.urdf.xacro (robot description, xacro)
@@ -1,4 +1,8 @@
 <?xml version='1.0' encoding='utf-8'?>
 <robot xmlns:xacro="http://www.ros.org/wiki/xacro" name="omniseer" xmlns:gz="http://gazebosim.org/schema">
+    <xacro:property name="min_vel" value="-50"/>
+    <xacro:property name="max_vel" value="50"/>
+    <xacro:property name="slip1" value="0.001"/>
+    <xacro:property name="slip2" value="0.001"/>
     <xacro:property name="kp"   value="1e5"/>
     <xacro:property name="kd"   value="1.0"/>
@@ -10,4 +14,5 @@
     <xacro:property name="ly" value="0.0866"/>
     <xacro:property name="wheel_radius" value="0.0485"/>
+    <xacro:property name="wheel_width" value="0.0445"/>
     <xacro:macro name="wheel_transmission" params="joint">
         <transmission name="${joint}_tr">
@@ -42,7 +47,8 @@
         </visual>
         <collision name="fl_wheel_collision">
-            <origin xyz="1.7993155232431945e-09 1.1387656346129211e-09 0.021000000766778337" rpy="1.5707963267948968 1.2281842209915656e-15 3.1554436208840444e-30" />
-            <geometry>
-                <mesh filename="package://omniseer_description/meshes/fl_wheel.stl" scale="0.001 0.001 0.001" />
+            <origin xyz="1.7993155232431945e-09 1.1387656346129211e-09 0.021000000766778337" rpy="0 1.2281842209915656e-15 3.1554436208840444e-30" />
+            <geometry>
+                <!-- <mesh filename="package://omniseer_description/meshes/fl_wheel.stl" scale="0.001 0.001 0.001" /> -->
+                <cylinder radius="${wheel_radius}" length="${wheel_width}"/>
             </geometry>
         </collision>
@@ -64,7 +70,8 @@
         </visual>
         <collision name="bl_wheel_collision">
-            <origin xyz="-1.7993151324446899e-09 1.1387656346129211e-09 0.021000000766778337" rpy="1.5707963267948968 1.2281842209915656e-15 3.1554436208840444e-30" />
-            <geometry>
-                <mesh filename="package://omniseer_description/meshes/bl_wheel.stl" scale="0.001 0.001 0.001" />
+            <origin xyz="-1.7993151324446899e-09 1.1387656346129211e-09 0.021000000766778337" rpy="0 1.2281842209915656e-15 3.1554436208840444e-30" />
+            <geometry>
+                <!-- <mesh filename="package://omniseer_description/meshes/bl_wheel.stl" scale="0.001 0.001 0.001" /> -->
+                <cylinder radius="${wheel_radius}" length="${wheel_width}"/>
             </geometry>
         </collision>
@@ -86,7 +93,8 @@
         </visual>
         <collision name="fr_wheel_collision">
-            <origin xyz="1.7993155765338997e-09 -1.1387656346129211e-09 0.02100000076677823" rpy="-1.5707963267948966 -1.2281842209915656e-15 -3.1554436208840444e-30" />
-            <geometry>
-                <mesh filename="package://omniseer_description/meshes/fr_wheel.stl" scale="0.001 0.001 0.001" />
+            <origin xyz="1.7993155765338997e-09 -1.1387656346129211e-09 0.02100000076677823" rpy="0 -1.2281842209915656e-15 -3.1554436208840444e-30" />
+            <geometry>
+                <!-- <mesh filename="package://omniseer_description/meshes/fr_wheel.stl" scale="0.001 0.001 0.001" /> -->
+                <cylinder radius="${wheel_radius}" length="${wheel_width}"/>
             </geometry>
         </collision>
@@ -108,7 +116,8 @@
         </visual>
         <collision name="br_wheel_collision">
-            <origin xyz="-1.7993150791539846e-09 -1.1387656346129211e-09 0.02100000076677823" rpy="-1.5707963267948966 -1.2281842209915656e-15 -3.1554436208840444e-30" />
-            <geometry>
-                <mesh filename="package://omniseer_description/meshes/br_wheel.stl" scale="0.001 0.001 0.001" />
+            <origin xyz="-1.7993150791539846e-09 -1.1387656346129211e-09 0.02100000076677823" rpy="0 -1.2281842209915656e-15 -3.1554436208840444e-30" />
+            <geometry>
+                <!-- <mesh filename="package://omniseer_description/meshes/br_wheel.stl" scale="0.001 0.001 0.001" /> -->
+                <cylinder radius="${wheel_radius}" length="${wheel_width}"/>
             </geometry>
         </collision>
@@ -163,4 +172,5 @@
         <child link="br_wheel" />
         <axis xyz="0.0 0.0 -1.0" />
+        <dynamics damping="0.1"/>
     </joint>
     <joint name="chassis_fr_wheel_joint" type="continuous">
@@ -169,4 +179,5 @@
         <child link="fr_wheel" />
         <axis xyz="-0.0 -0.0 -1.0" />
+        <dynamics damping="0.1"/>
     </joint>
     <joint name="chassis_bl_wheel_joint" type="continuous">
@@ -175,4 +186,5 @@
         <child link="bl_wheel" />
         <axis xyz="0.0 0.0 1.0" />
+        <dynamics damping="0.1"/>
     </joint>
     <joint name="chassis_fl_wheel_joint" type="continuous">
@@ -181,4 +193,5 @@
         <child link="fl_wheel" />
         <axis xyz="0.0 0.0 1.0" />
+        <dynamics damping="0.1"/>
     </joint>
     <joint name="chassis_lidar_joint" type="fixed">
@@ -199,6 +212,6 @@
         <joint name="chassis_fl_wheel_joint">
             <command_interface name="velocity">
-                <param name="min">-10</param>
-                <param name="max">10</param>
+                <param name="min">${min_vel}</param>
+                <param name="max">${max_vel}</param>
             </command_interface>
             <state_interface   name="velocity"/>
@@ -208,6 +221,6 @@
         <joint name="chassis_fr_wheel_joint">
             <command_interface name="velocity">
-                <param name="min">-10</param>
-                <param name="max">10</param>
+                <param name="min">${min_vel}</param>
+                <param name="max">${max_vel}</param>
             </command_interface>
             <state_interface   name="velocity"/>
@@ -217,6 +230,6 @@
         <joint name="chassis_bl_wheel_joint">
             <command_interface name="velocity">
-                <param name="min">-10</param>
-                <param name="max">10</param>
+                <param name="min">${min_vel}</param>
+                <param name="max">${max_vel}</param>
             </command_interface>
             <state_interface   name="velocity"/>
@@ -226,6 +239,6 @@
         <joint name="chassis_br_wheel_joint">
             <command_interface name="velocity">
-                <param name="min">-10</param>
-                <param name="max">10</param>
+                <param name="min">${min_vel}</param>
+                <param name="max">${max_vel}</param>
             </command_interface>
             <state_interface   name="velocity"/>
@@ -241,4 +254,6 @@
                         <mu>${mu}</mu>
                         <mu2>${mu2}</mu2>
+                        <slip1>${slip1}</slip1>
+                        <slip2>${slip2}</slip2>
                         <fdir1 gz:expressed_in="base_link">1 -1 0</fdir1>
                     </ode>
@@ -260,4 +275,6 @@
                     <mu>${mu}</mu>
                     <mu2>${mu2}</mu2>
+                    <slip1>${slip1}</slip1>
+                    <slip2>${slip2}</slip2>
                     <fdir1 gz:expressed_in="base_link">1 1 0</fdir1>
                 </ode>
@@ -279,4 +296,6 @@
                         <mu>${mu}</mu>
                         <mu2>${mu2}</mu2>
+                        <slip1>${slip1}</slip1>
+                        <slip2>${slip2}</slip2>
                         <fdir1 gz:expressed_in="base_link">1 1 0</fdir1>
                     </ode>
@@ -298,4 +317,6 @@
                         <mu>${mu}</mu>
                         <mu2>${mu2}</mu2>
+                        <slip1>${slip1}</slip1>
+                        <slip2>${slip2}</slip2>
                         <fdir1 gz:expressed_in="base_link">1 -1 0</fdir1>
                     </ode>

Commit message: feat: lidar integrated and confirmed working via RVIZ laserscan, rviz config updates.

File: ros_ws/src/omniseer_description/urdf/xacro/omniseer.urdf.xacro (robot description, xacro)
@@ -10,5 +10,6 @@
     <xacro:property name="mu2"   value="0.05"/>
     <xacro:property name="body_rgba"   value="0.671 0.663 0.506 1.0"/>
-    <xacro:property name="sensor_rgba" value="0.0 0.0 0.0 1.0"/>
+    <xacro:property name="sensor_rgba" value="0.671 0.663 0.506 1.0"/>
+    <xacro:property name="debug_rgba" value="1.0 0.0 0.0 1.0"/>
     <xacro:property name="lx" value="0.0974"/>
     <xacro:property name="ly" value="0.0866"/>
@@ -146,4 +147,7 @@
     </link>
     <link name="lidar_top">
+        <frame name="lidar_frame" attached_to="lidar_top">
+            <pose>0 0 -0.076 0 0 0</pose>
+        </frame>
         <inertial>
             <origin xyz="-2.954093418429609e-17 9.748508280817712e-16 0.009999998873493041" rpy="0.0 -0.0 0.0" />
@@ -167,4 +171,34 @@
         </collision>
     </link>
+    <link name="lidar_frame"/>
+    <link name="imu_link">
+        <inertial>
+            <origin xyz="0 0 0" rpy="0 0 0"/>
+            <mass value="0.01"/>
+            <inertia
+                ixx="1e-7" ixy="0.0" ixz="0.0"
+                iyy="1e-7" iyz="0.0"
+                izz="1e-7"/>
+        </inertial>
+        <!-- no collision/visual required -->
+        <visual name="imu_viz">
+            <!-- <geometry><box size="0.01 0.01 0.003"/></geometry> -->
+            <geometry><box size="0.01 0.01 0.01"/></geometry>
+            <material name='r'>
+                <color rgba="${debug_rgba}"/>
+            </material>
+        </visual>
+    </link>
+    <joint name="lidar_top_to_frame" type="fixed">
+        <parent link="lidar_top"/>
+        <child  link="lidar_frame"/>
+        <!-- offset halfway up the cylinder -->
+        <origin xyz="0 0 -0.076" rpy="0 0 0"/>
+    </joint>
+    <joint name="chassis_imu_joint" type="fixed">
+        <parent link="chassis"/>
+        <child  link="imu_link"/>
+        <origin xyz="0.01 0 0.045" rpy="0 0 0"/>
+    </joint>
     <joint name="chassis_br_wheel_joint" type="continuous">
         <origin xyz="-0.0971 -0.08661705 8.94e-06" rpy="1.5707963267948966 -0.0 0.0" />
@@ -247,4 +281,50 @@
         </joint>
     </ros2_control>
+    <gazebo reference="lidar_top">
+        <sensor name="rplidar_a1" type="gpu_lidar">
+            <frame_id>lidar_frame</frame_id>
+            <pose>0 0 0 0 0 0</pose>
+            <topic>lidar</topic>
+            <update_rate>10</update_rate>
+            <ray>
+                <scan>
+                    <horizontal>
+                    <samples>360</samples>
+                    <resolution>1</resolution>
+                    <min_angle>-3.14159</min_angle>
+                    <max_angle> 3.14159</max_angle>
+                    </horizontal>
+                </scan>
+                <range>
+                    <min>0.12</min>
+                    <max>12.0</max>
+                    <resolution>0.01</resolution>
+                </range>
+            </ray>
+            <always_on>1</always_on>
+            <visualize>true</visualize>
+        </sensor>
+    </gazebo>
+    <gazebo reference="imu_link">
+        <sensor name="imu_sensor" type="imu">
+            <pose>0 0 0 0 0 0</pose>
+            <always_on>1</always_on>
+            <update_rate>200</update_rate>
+            <topic>imu</topic>
+            <imu>
+                <!-- <orientation_reference_frame>ENU</orientation_reference_frame> -->
+                <angular_velocity>
+                    <x><noise type="gaussian"><mean>0</mean><stddev>0.001</stddev></noise></x>
+                    <y><noise type="gaussian"><mean>0</mean><stddev>0.001</stddev></noise></y>
+                    <z><noise type="gaussian"><mean>0</mean><stddev>0.001</stddev></noise></z>
+                </angular_velocity>
+                <linear_acceleration>
+                    <x><noise type="gaussian"><mean>0</mean><stddev>0.10</stddev></noise></x>
+                    <y><noise type="gaussian"><mean>0</mean><stddev>0.10</stddev></noise></y>
+                    <z><noise type="gaussian"><mean>0</mean><stddev>0.10</stddev></noise></z>
+                </linear_acceleration>
+            </imu>
+        </sensor>
+    </gazebo>
     <gazebo reference='fl_wheel'>
         <collision>
@@ -341,9 +421,9 @@
     </gazebo>
     <gazebo>
-        <plugin filename="gz-sim-odometry-publisher-system" name="gz::sim::systems::OdometryPublisher">
+        <plugin name="gz::sim::systems::OdometryPublisher" filename="gz-sim-odometry-publisher-system">
             <dimensions>3</dimensions>
             <odom_publish_frequency>50</odom_publish_frequency>
+            <odom_topic>/model_odom</odom_topic>
             <odom_frame>odom</odom_frame>
-            <odom_topic>/model_odom</odom_topic>
             <robot_base_frame>base_link</robot_base_frame>
         </plugin>

Commit message: feat: sonar operational, publishing on /range

File: ros_ws/src/omniseer_description/urdf/xacro/omniseer.urdf.xacro (robot description, xacro)
@@ -32,4 +32,5 @@
     <xacro:wheel_transmission joint="chassis_bl_wheel_joint"/>
     <xacro:wheel_transmission joint="chassis_br_wheel_joint"/>
+    <!-- Links -->
     <link name="fl_wheel">
         <inertial>
@@ -50,5 +51,4 @@
             <origin xyz="1.7993155232431945e-09 1.1387656346129211e-09 0.021000000766778337" rpy="0 1.2281842209915656e-15 3.1554436208840444e-30" />
             <geometry>
-                <!-- <mesh filename="package://omniseer_description/meshes/fl_wheel.stl" scale="0.001 0.001 0.001" /> -->
                 <cylinder radius="${wheel_radius}" length="${wheel_width}"/>
             </geometry>
@@ -73,5 +73,4 @@
             <origin xyz="-1.7993151324446899e-09 1.1387656346129211e-09 0.021000000766778337" rpy="0 1.2281842209915656e-15 3.1554436208840444e-30" />
             <geometry>
-                <!-- <mesh filename="package://omniseer_description/meshes/bl_wheel.stl" scale="0.001 0.001 0.001" /> -->
                 <cylinder radius="${wheel_radius}" length="${wheel_width}"/>
             </geometry>
@@ -96,5 +95,4 @@
             <origin xyz="1.7993155765338997e-09 -1.1387656346129211e-09 0.02100000076677823" rpy="0 -1.2281842209915656e-15 -3.1554436208840444e-30" />
             <geometry>
-                <!-- <mesh filename="package://omniseer_description/meshes/fr_wheel.stl" scale="0.001 0.001 0.001" /> -->
                 <cylinder radius="${wheel_radius}" length="${wheel_width}"/>
             </geometry>
@@ -119,5 +117,4 @@
             <origin xyz="-1.7993150791539846e-09 -1.1387656346129211e-09 0.02100000076677823" rpy="0 -1.2281842209915656e-15 -3.1554436208840444e-30" />
             <geometry>
-                <!-- <mesh filename="package://omniseer_description/meshes/br_wheel.stl" scale="0.001 0.001 0.001" /> -->
                 <cylinder radius="${wheel_radius}" length="${wheel_width}"/>
             </geometry>
@@ -172,5 +169,5 @@
     </link>
     <link name="lidar_frame"/>
-    <link name="imu_link">
+    <link name="sonar_link">
         <inertial>
             <origin xyz="0 0 0" rpy="0 0 0"/>
@@ -181,7 +178,5 @@
                 izz="1e-7"/>
         </inertial>
-        <!-- no collision/visual required -->
-        <visual name="imu_viz">
-            <!-- <geometry><box size="0.01 0.01 0.003"/></geometry> -->
+        <visual name="sonar_viz">
             <geometry><box size="0.01 0.01 0.01"/></geometry>
             <material name='r'>
@@ -190,8 +185,29 @@
         </visual>
     </link>
+    <link name="imu_link">
+        <inertial>
+            <origin xyz="0 0 0" rpy="0 0 0"/>
+            <mass value="0.01"/>
+            <inertia
+                ixx="1e-7" ixy="0.0" ixz="0.0"
+                iyy="1e-7" iyz="0.0"
+                izz="1e-7"/>
+        </inertial>
+        <visual name="imu_viz">
+            <geometry><box size="0.01 0.01 0.01"/></geometry>
+            <material name='r'>
+                <color rgba="${debug_rgba}"/>
+            </material>
+        </visual>
+    </link>
+    <!-- Joints -->
+    <joint name="chassis_sonar_joint" type="fixed">
+        <parent link="chassis"/>
+        <child  link="sonar_link"/>
+        <origin xyz="0.1775 0 0.015" rpy="0 0 0"/>
+    </joint>
     <joint name="lidar_top_to_frame" type="fixed">
         <parent link="lidar_top"/>
         <child  link="lidar_frame"/>
-        <!-- offset halfway up the cylinder -->
         <origin xyz="0 0 -0.076" rpy="0 0 0"/>
     </joint>
@@ -281,4 +297,29 @@
         </joint>
     </ros2_control>
+    <!-- Gazebo -->
+    <gazebo reference="sonar_link">
+        <sensor name="sonar" type="gpu_lidar">
+            <frame_id>sonar_link</frame_id>
+            <pose>0 0 0 0 0 0</pose>
+            <update_rate>20</update_rate>
+            <topic>sonar</topic>
+            <ray>
+                <scan>
+                    <horizontal>
+                        <samples>21</samples>
+                        <min_angle>-0.131</min_angle>
+                        <max_angle> 0.131</max_angle>
+                    </horizontal>
+                </scan>
+                <range>
+                    <min>0.02</min>
+                    <max>4.0</max>
+                    <resolution>0.01</resolution>
+                </range>
+            </ray>
+            <always_on>1</always_on>
+            <visualize>true</visualize>
+        </sensor>
+    </gazebo>
     <gazebo reference="lidar_top">
         <sensor name="rplidar_a1" type="gpu_lidar">
@@ -313,5 +354,4 @@
             <topic>imu</topic>
             <imu>
-                <!-- <orientation_reference_frame>ENU</orientation_reference_frame> -->
                 <angular_velocity>
                     <x><noise type="gaussian"><mean>0</mean><stddev>0.001</stddev></noise></x>

Commit message: feat: pre flight gz cleanup, nodes are separate OS processes, no killall exists

File: ros_ws/src/omniseer_description/urdf/xacro/omniseer.urdf.xacro (robot description, xacro)
@@ -201,5 +201,26 @@
         </visual>
     </link>
+    <link name="camera_link">
+        <inertial>
+            <origin xyz="0 0 0" rpy="0 0 0"/>
+            <mass value="0.01"/>
+            <inertia
+                ixx="1e-7" ixy="0.0" ixz="0.0"
+                iyy="1e-7" iyz="0.0"
+                izz="1e-7"/>
+        </inertial>
+        <visual name="camera_viz">
+            <geometry><box size="0.01 0.01 0.01"/></geometry>
+            <material name='r'>
+                <color rgba="${debug_rgba}"/>
+            </material>
+        </visual>
+    </link>
     <!-- Joints -->
+    <joint name="chassis_camera_joint" type="fixed">
+        <parent link="chassis"/>
+        <child  link="camera_link"/>
+        <origin xyz="0.145 0.0 0.1248" rpy="0 0 0"/>
+    </joint>
     <joint name="chassis_sonar_joint" type="fixed">
         <parent link="chassis"/>
@@ -298,4 +319,24 @@
     </ros2_control>
     <!-- Gazebo -->
+    <gazebo reference="camera_link">
+        <sensor name="front_camera" type="camera">
+            <update_rate>30</update_rate>
+            <always_on>1</always_on>
+            <topic>front_camera/image</topic>
+            <camera>
+                <horizontal_fov>1.309</horizontal_fov>
+                <image>
+                    <width>1920</width>
+                    <height>1080</height>
+                    <format>R8G8B8</format>
+                </image>
+                <clip>
+                    <near>0.03</near>
+                    <far>100</far>
+                </clip>
+            </camera>
+            <visualize>true</visualize>
+        </sensor>
+    </gazebo>
     <gazebo reference="sonar_link">
         <sensor name="sonar" type="gpu_lidar">
