Commit message: refactor(launch) + feat(ekf): orchestrate_sim.launch, modular bringup. sensor fusion imu+encoder, tuned to sim

File: ros_ws/src/omniseer_description/urdf/xacro/omniseer.urdf.xacro (robot description, xacro)
@@ -12,6 +12,4 @@
     <xacro:property name="sensor_rgba" value="0.671 0.663 0.506 1.0"/>
     <xacro:property name="debug_rgba" value="1.0 0.0 0.0 1.0"/>
-    <xacro:property name="lx" value="0.0974"/>
-    <xacro:property name="ly" value="0.0866"/>
     <xacro:property name="wheel_radius" value="0.0485"/>
     <xacro:property name="wheel_width" value="0.0445"/>
@@ -35,10 +33,10 @@
     <link name="fl_wheel">
         <inertial>
-            <origin xyz="1.7993153278439422e-09 2.26380317489938e-09 0.02100000076677828" rpy="0.0 -0.0 0.0" />
+            <origin xyz="1.7993153278439422e-09 0 0" rpy="0.0 -0.0 0.0" />
             <mass value="0.1449437592188408" />
             <inertia ixx="0.00010654272201079539" iyy="0.00010654272201080037" izz="0.00017047197881125639" ixy="-4.7460314825842516e-20" iyz="-5.1880768019325896e-20" ixz="0.0" />
         </inertial>
         <visual name="fl_wheel_visual">
-            <origin xyz="1.7993155232431945e-09 1.1387656346129211e-09 0.021000000766778337" rpy="1.5707963267948968 1.2281842209915656e-15 3.1554436208840444e-30" />
+            <origin xyz="1.7993155232431945e-09 0 0" rpy="1.5707963267948968 1.2281842209915656e-15 3.1554436208840444e-30" />
             <geometry>
                 <mesh filename="package://omniseer_description/meshes/fl_wheel.stl" scale="0.001 0.001 0.001" />
@@ -49,5 +47,5 @@
         </visual>
         <collision name="fl_wheel_collision">
-            <origin xyz="1.7993155232431945e-09 1.1387656346129211e-09 0.021000000766778337" rpy="0 1.2281842209915656e-15 3.1554436208840444e-30" />
+            <origin xyz="1.7993155232431945e-09 0 0" rpy="0 1.2281842209915656e-15 3.1554436208840444e-30" />
             <geometry>
                 <cylinder radius="${wheel_radius}" length="${wheel_width}"/>
@@ -57,10 +55,10 @@
     <link name="bl_wheel">
         <inertial>
-            <origin xyz="-1.7993153278439422e-09 2.26380317489938e-09 0.02100000076677828" rpy="0.0 -0.0 0.0" />
+            <origin xyz="-1.7993153278439422e-09 0 0" rpy="0.0 -0.0 0.0" />
             <mass value="0.1449437592188408" />
             <inertia ixx="0.00010654272201079539" iyy="0.0001065427220107995" izz="0.00017047197881125617" ixy="-4.7460314825842516e-20" iyz="-5.1880768019325896e-20" ixz="0.0" />
         </inertial>
         <visual name="bl_wheel_visual">
-            <origin xyz="-1.7993151324446899e-09 1.1387656346129211e-09 0.021000000766778337" rpy="1.5707963267948968 1.2281842209915656e-15 3.1554436208840444e-30" />
+            <origin xyz="-1.7993151324446899e-09 0 0" rpy="1.5707963267948968 1.2281842209915656e-15 3.1554436208840444e-30" />
             <geometry>
                 <mesh filename="package://omniseer_description/meshes/bl_wheel.stl" scale="0.001 0.001 0.001" />
@@ -71,5 +69,5 @@
         </visual>
         <collision name="bl_wheel_collision">
-            <origin xyz="-1.7993151324446899e-09 1.1387656346129211e-09 0.021000000766778337" rpy="0 1.2281842209915656e-15 3.1554436208840444e-30" />
+            <origin xyz="-1.7993151324446899e-09 0 0" rpy="0 1.2281842209915656e-15 3.1554436208840444e-30" />
             <geometry>
                 <cylinder radius="${wheel_radius}" length="${wheel_width}"/>
@@ -79,10 +77,10 @@
     <link name="fr_wheel">
         <inertial>
-            <origin xyz="1.7993153811346474e-09 -2.26380317489938e-09 0.02100000076677828" rpy="0.0 -0.0 0.0" />
+            <origin xyz="1.7993153811346474e-09 0.0 -0" rpy="0.0 -0.0 0.0" />
             <mass value="0.1449437592188408" />
             <inertia ixx="0.00010654272201079539" iyy="0.00010654272201079994" izz="0.00017047197881125639" ixy="4.7460314825842516e-20" iyz="-5.1880768019325896e-20" ixz="0.0" />
         </inertial>
         <visual name="fr_wheel_visual">
-            <origin xyz="1.7993155765338997e-09 -1.1387656346129211e-09 0.02100000076677823" rpy="-1.5707963267948966 -1.2281842209915656e-15 -3.1554436208840444e-30" />
+            <origin xyz="1.7993155765338997e-09 0 -0" rpy="-1.5707963267948966 -1.2281842209915656e-15 -3.1554436208840444e-30" />
             <geometry>
                 <mesh filename="package://omniseer_description/meshes/fr_wheel.stl" scale="0.001 0.001 0.001" />
@@ -93,5 +91,5 @@
         </visual>
         <collision name="fr_wheel_collision">
-            <origin xyz="1.7993155765338997e-09 -1.1387656346129211e-09 0.02100000076677823" rpy="0 -1.2281842209915656e-15 -3.1554436208840444e-30" />
+            <origin xyz="1.7993155765338997e-09 0 -0" rpy="0 -1.2281842209915656e-15 -3.1554436208840444e-30" />
             <geometry>
                 <cylinder radius="${wheel_radius}" length="${wheel_width}"/>
@@ -101,10 +99,10 @@
     <link name="br_wheel">
         <inertial>
-            <origin xyz="-1.7993152745532372e-09 -2.26380317489938e-09 0.02100000076677828" rpy="0.0 -0.0 0.0" />
+            <origin xyz="-1.7993152745532372e-09 0 -0" rpy="0.0 -0.0 0.0" />
             <mass value="0.1449437592188408" />
             <inertia ixx="0.00010654272201079539" iyy="0.00010654272201080037" izz="0.00017047197881125617" ixy="4.7460314825842516e-20" iyz="-5.1880768019325896e-20" ixz="-4.336808689942018e-19" />
         </inertial>
         <visual name="br_wheel_visual">
-            <origin xyz="-1.7993150791539846e-09 -1.1387656346129211e-09 0.02100000076677823" rpy="-1.5707963267948966 -1.2281842209915656e-15 -3.1554436208840444e-30" />
+            <origin xyz="-1.7993150791539846e-09 0 -0" rpy="-1.5707963267948966 -1.2281842209915656e-15 -3.1554436208840444e-30" />
             <geometry>
                 <mesh filename="package://omniseer_description/meshes/br_wheel.stl" scale="0.001 0.001 0.001" />
@@ -115,5 +113,5 @@
         </visual>
         <collision name="br_wheel_collision">
-            <origin xyz="-1.7993150791539846e-09 -1.1387656346129211e-09 0.02100000076677823" rpy="0 -1.2281842209915656e-15 -3.1554436208840444e-30" />
+            <origin xyz="-1.7993150791539846e-09 0 -0" rpy="0 -1.2281842209915656e-15 -3.1554436208840444e-30" />
             <geometry>
                 <cylinder radius="${wheel_radius}" length="${wheel_width}"/>
@@ -239,5 +237,5 @@
     </joint>
     <joint name="chassis_br_wheel_joint" type="continuous">
-        <origin xyz="-0.0971 -0.08661705 8.94e-06" rpy="1.5707963267948966 -0.0 0.0" />
+        <origin xyz="-0.0971 -0.10886705 8.94e-06" rpy="1.5707963267948966 -0.0 0.0" />
         <parent link="chassis" />
         <child link="br_wheel" />
@@ -246,5 +244,5 @@
     </joint>
     <joint name="chassis_fr_wheel_joint" type="continuous">
-        <origin xyz="0.0976 -0.08661705 8.94e-06" rpy="1.5707963267948966 -0.0 0.0" />
+        <origin xyz="0.0976 -0.10886705 8.94e-06" rpy="1.5707963267948966 -0.0 0.0" />
         <parent link="chassis" />
         <child link="fr_wheel" />
@@ -253,5 +251,5 @@
     </joint>
     <joint name="chassis_bl_wheel_joint" type="continuous">
-        <origin xyz="-0.0971 0.08661705 8.94e-06" rpy="-1.5707963267948966 -0.0 0.0" />
+        <origin xyz="-0.0971 0.10886705 8.94e-06" rpy="-1.5707963267948966 -0.0 0.0" />
         <parent link="chassis" />
         <child link="bl_wheel" />
@@ -260,5 +258,5 @@
     </joint>
     <joint name="chassis_fl_wheel_joint" type="continuous">
-        <origin xyz="0.0976 0.08661705 8.94e-06" rpy="-1.5707963267948966 -0.0 0.0" />
+        <origin xyz="0.0976 0.10886705 8.94e-06" rpy="-1.5707963267948966 -0.0 0.0" />
         <parent link="chassis" />
         <child link="fl_wheel" />
@@ -390,4 +388,5 @@
     <gazebo reference="imu_link">
         <sensor name="imu_sensor" type="imu">
+            <frame_id>imu_link</frame_id>
             <pose>0 0 0 0 0 0</pose>
             <always_on>1</always_on>
@@ -495,7 +494,6 @@
         <plugin name="gz_ros2_control::GazeboSimROS2ControlPlugin" filename="libgz_ros2_control-system">
             <verbose>true</verbose>
-            <parameters>
-                $(find bringup)/config/controllers.yaml
-            </parameters>
+            <parameters>$(find bringup)/config/controllers.yaml</parameters>
+            <param name="config_file" value="$(find bringup)/config/controllers.yaml"/>
             <controller_manager_prefix_node_name>controller_manager</controller_manager_prefix_node_name>
         </plugin>

Commit message: feat(nav2, rf2o)/refactor(launch): container runs OpenGL / CUDA, launch hardened. rf2o ekf

File: ros_ws/src/omniseer_description/urdf/xacro/omniseer.urdf.xacro (robot description, xacro)
@@ -14,20 +14,4 @@
     <xacro:property name="wheel_radius" value="0.0485"/>
     <xacro:property name="wheel_width" value="0.0445"/>
-    <xacro:macro name="wheel_transmission" params="joint">
-        <transmission name="${joint}_tr">
-            <type>transmission_interface/SimpleTransmission</type>
-            <joint name="${joint}">
-                <hardwareInterface>hardware_interface/VelocityJointInterface</hardwareInterface>
-            </joint>
-            <actuator name="${joint}_motor">
-                <hardwareInterface>hardware_interface/VelocityJointInterface</hardwareInterface>
-                <mechanicalReduction>1</mechanicalReduction>
-            </actuator>
-        </transmission>
-    </xacro:macro>
-    <xacro:wheel_transmission joint="chassis_fl_wheel_joint"/>
-    <xacro:wheel_transmission joint="chassis_fr_wheel_joint"/>
-    <xacro:wheel_transmission joint="chassis_bl_wheel_joint"/>
-    <xacro:wheel_transmission joint="chassis_br_wheel_joint"/>
     <!-- Links -->
     <link name="fl_wheel">
@@ -141,4 +125,5 @@
         </collision>
     </link>
+    <link name="lidar_frame"/>
     <link name="lidar_top">
         <frame name="lidar_frame" attached_to="lidar_top">
@@ -166,5 +151,4 @@
         </collision>
     </link>
-    <link name="lidar_frame"/>
     <link name="sonar_link">
         <inertial>
@@ -365,5 +349,5 @@
             <frame_id>lidar_frame</frame_id>
             <pose>0 0 0 0 0 0</pose>
-            <topic>lidar</topic>
+            <topic>scan</topic>
             <update_rate>10</update_rate>
             <ray>
@@ -495,5 +479,4 @@
             <verbose>true</verbose>
             <parameters>$(find bringup)/config/controllers.yaml</parameters>
-            <param name="config_file" value="$(find bringup)/config/controllers.yaml"/>
             <controller_manager_prefix_node_name>controller_manager</controller_manager_prefix_node_name>
         </plugin>

Commit message: refactor(Dockerfile): fully audited Dockerfile, application is now fully reproducible on ubunutu/nvidia box. can teleoperate robot in sim, YOLO-World detector functioning

File: ros_ws/src/omniseer_description/urdf/xacro/omniseer.urdf.xacro (robot description, xacro)
@@ -24,5 +24,5 @@
             <origin xyz="1.7993155232431945e-09 0 0" rpy="1.5707963267948968 1.2281842209915656e-15 3.1554436208840444e-30" />
             <geometry>
-                <mesh filename="package://omniseer_description/meshes/fl_wheel.stl" scale="0.001 0.001 0.001" />
+                <mesh filename="file://$(find omniseer_description)/meshes/fl_wheel.stl" scale="0.001 0.001 0.001"/>
             </geometry>
             <material name='body_mat'>
@@ -46,5 +46,5 @@
             <origin xyz="-1.7993151324446899e-09 0 0" rpy="1.5707963267948968 1.2281842209915656e-15 3.1554436208840444e-30" />
             <geometry>
-                <mesh filename="package://omniseer_description/meshes/bl_wheel.stl" scale="0.001 0.001 0.001" />
+                <mesh filename="file://$(find omniseer_description)/meshes/bl_wheel.stl" scale="0.001 0.001 0.001"/>
             </geometry>
             <material name='body_mat'>
@@ -68,5 +68,5 @@
             <origin xyz="1.7993155765338997e-09 0 -0" rpy="-1.5707963267948966 -1.2281842209915656e-15 -3.1554436208840444e-30" />
             <geometry>
-                <mesh filename="package://omniseer_description/meshes/fr_wheel.stl" scale="0.001 0.001 0.001" />
+                <mesh filename="file://$(find omniseer_description)/meshes/fr_wheel.stl" scale="0.001 0.001 0.001"/>
             </geometry>
             <material name='body_mat'>
@@ -90,5 +90,5 @@
             <origin xyz="-1.7993150791539846e-09 0 -0" rpy="-1.5707963267948966 -1.2281842209915656e-15 -3.1554436208840444e-30" />
             <geometry>
-                <mesh filename="package://omniseer_description/meshes/br_wheel.stl" scale="0.001 0.001 0.001" />
+                <mesh filename="file://$(find omniseer_description)/meshes/br_wheel.stl" scale="0.001 0.001 0.001"/>
             </geometry>
             <material name='body_mat'>
@@ -112,5 +112,5 @@
             <origin xyz="0.0 0.0 0.0" rpy="0.0 0.0 0.0" />
             <geometry>
-                <mesh filename="package://omniseer_description/meshes/chassis.stl" scale="0.001 0.001 0.001" />
+                <mesh filename="file://$(find omniseer_description)/meshes/chassis.stl" scale="0.001 0.001 0.001"/>
             </geometry>
             <material name='body_mat'>
@@ -121,5 +121,5 @@
             <origin xyz="0.0 0.0 0.0" rpy="0.0 0.0 0.0" />
             <geometry>
-                <mesh filename="package://omniseer_description/meshes/chassis.stl" scale="0.001 0.001 0.001" />
+                <mesh filename="file://$(find omniseer_description)/meshes/chassis.stl" scale="0.001 0.001 0.001"/>
             </geometry>
         </collision>
@@ -138,5 +138,5 @@
             <origin xyz="0.0 0.0 -0.15209671" rpy="0.0 -0.0 0.0" />
             <geometry>
-                <mesh filename="package://omniseer_description/meshes/lidar_top.stl" scale="0.001 0.001 0.001" />
+                <mesh filename="file://$(find omniseer_description)/meshes/lidar_top.stl" scale="0.001 0.001 0.001"/>
             </geometry>
             <material name='sensor_mat'>
@@ -147,5 +147,5 @@
             <origin xyz="0.0 0.0 -0.15209671" rpy="0.0 -0.0 0.0" />
             <geometry>
-                <mesh filename="package://omniseer_description/meshes/lidar_top.stl" scale="0.001 0.001 0.001" />
+                <mesh filename="file://$(find omniseer_description)/meshes/lidar_top.stl" scale="0.001 0.001 0.001"/>
             </geometry>
         </collision>

Commit message: refactor(bringup): split shared, sim, and real launch layers around the IO boundary.

File: ros_ws/src/omniseer_description/urdf/xacro/omniseer.urdf.xacro (robot description, xacro)
@@ -1,4 +1,6 @@
 <?xml version='1.0' encoding='utf-8'?>
 <robot xmlns:xacro="http://www.ros.org/wiki/xacro" name="omniseer" xmlns:gz="http://gazebosim.org/schema">
+    <xacro:arg name="use_ci_geometry" default="false"/>
+    <xacro:property name="use_ci_geometry" value="$(arg use_ci_geometry)"/>
     <xacro:property name="min_vel" value="-50"/>
     <xacro:property name="max_vel" value="50"/>
@@ -110,7 +112,11 @@
         </inertial>
         <visual name="chassis_visual">
-            <origin xyz="0.0 0.0 0.0" rpy="0.0 0.0 0.0" />
-            <geometry>
-                <mesh filename="file://$(find omniseer_description)/meshes/chassis.stl" scale="0.001 0.001 0.001"/>
+            <geometry>
+                <xacro:if value="${use_ci_geometry}">
+                    <box size="0.28 0.23 0.11"/>
+                </xacro:if>
+                <xacro:unless value="${use_ci_geometry}">
+                    <mesh filename="file://$(find omniseer_description)/meshes/chassis.stl" scale="0.001 0.001 0.001"/>
+                </xacro:unless>
             </geometry>
             <material name='body_mat'>
@@ -119,7 +125,11 @@
         </visual>
         <collision name="chassis_collision">
-            <origin xyz="0.0 0.0 0.0" rpy="0.0 0.0 0.0" />
-            <geometry>
-                <mesh filename="file://$(find omniseer_description)/meshes/chassis.stl" scale="0.001 0.001 0.001"/>
+            <geometry>
+                <xacro:if value="${use_ci_geometry}">
+                    <box size="0.28 0.23 0.11"/>
+                </xacro:if>
+                <xacro:unless value="${use_ci_geometry}">
+                    <mesh filename="file://$(find omniseer_description)/meshes/chassis.stl" scale="0.001 0.001 0.001"/>
+                </xacro:unless>
             </geometry>
         </collision>
@@ -136,7 +146,11 @@
         </inertial>
         <visual name="lidar_top_visual">
-            <origin xyz="0.0 0.0 -0.15209671" rpy="0.0 -0.0 0.0" />
-            <geometry>
-                <mesh filename="file://$(find omniseer_description)/meshes/lidar_top.stl" scale="0.001 0.001 0.001"/>
+            <geometry>
+                <xacro:if value="${use_ci_geometry}">
+                    <cylinder radius="0.045" length="0.03"/>
+                </xacro:if>
+                <xacro:unless value="${use_ci_geometry}">
+                    <mesh filename="file://$(find omniseer_description)/meshes/lidar_top.stl" scale="0.001 0.001 0.001"/>
+                </xacro:unless>
             </geometry>
             <material name='sensor_mat'>
@@ -145,7 +159,11 @@
         </visual>
         <collision name="lidar_top_collision">
-            <origin xyz="0.0 0.0 -0.15209671" rpy="0.0 -0.0 0.0" />
-            <geometry>
-                <mesh filename="file://$(find omniseer_description)/meshes/lidar_top.stl" scale="0.001 0.001 0.001"/>
+            <geometry>
+                <xacro:if value="${use_ci_geometry}">
+                    <cylinder radius="0.045" length="0.03"/>
+                </xacro:if>
+                <xacro:unless value="${use_ci_geometry}">
+                    <mesh filename="file://$(find omniseer_description)/meshes/lidar_top.stl" scale="0.001 0.001 0.001"/>
+                </xacro:unless>
             </geometry>
         </collision>
