Commit message: fix(bringup): serve RViz package resources

File: ros_ws/src/omniseer_description/urdf/xacro/omniseer.urdf.xacro (robot description, xacro)
@@ -26,5 +26,5 @@
             <origin xyz="1.7993155232431945e-09 0 0" rpy="1.5707963267948968 1.2281842209915656e-15 3.1554436208840444e-30" />
             <geometry>
-                <mesh filename="file://$(find omniseer_description)/meshes/fl_wheel.stl" scale="0.001 0.001 0.001"/>
+                <mesh filename="package://omniseer_description/meshes/fl_wheel.stl" scale="0.001 0.001 0.001"/>
             </geometry>
             <material name='body_mat'>
@@ -48,5 +48,5 @@
             <origin xyz="-1.7993151324446899e-09 0 0" rpy="1.5707963267948968 1.2281842209915656e-15 3.1554436208840444e-30" />
             <geometry>
-                <mesh filename="file://$(find omniseer_description)/meshes/bl_wheel.stl" scale="0.001 0.001 0.001"/>
+                <mesh filename="package://omniseer_description/meshes/bl_wheel.stl" scale="0.001 0.001 0.001"/>
             </geometry>
             <material name='body_mat'>
@@ -70,5 +70,5 @@
             <origin xyz="1.7993155765338997e-09 0 -0" rpy="-1.5707963267948966 -1.2281842209915656e-15 -3.1554436208840444e-30" />
             <geometry>
-                <mesh filename="file://$(find omniseer_description)/meshes/fr_wheel.stl" scale="0.001 0.001 0.001"/>
+                <mesh filename="package://omniseer_description/meshes/fr_wheel.stl" scale="0.001 0.001 0.001"/>
             </geometry>
             <material name='body_mat'>
@@ -92,5 +92,5 @@
             <origin xyz="-1.7993150791539846e-09 0 -0" rpy="-1.5707963267948966 -1.2281842209915656e-15 -3.1554436208840444e-30" />
             <geometry>
-                <mesh filename="file://$(find omniseer_description)/meshes/br_wheel.stl" scale="0.001 0.001 0.001"/>
+                <mesh filename="package://omniseer_description/meshes/br_wheel.stl" scale="0.001 0.001 0.001"/>
             </geometry>
             <material name='body_mat'>
@@ -117,5 +117,5 @@
                 </xacro:if>
                 <xacro:unless value="${use_ci_geometry}">
-                    <mesh filename="file://$(find omniseer_description)/meshes/chassis.stl" scale="0.001 0.001 0.001"/>
+                    <mesh filename="package://omniseer_description/meshes/chassis.stl" scale="0.001 0.001 0.001"/>
                 </xacro:unless>
             </geometry>
@@ -130,5 +130,5 @@
                 </xacro:if>
                 <xacro:unless value="${use_ci_geometry}">
-                    <mesh filename="file://$(find omniseer_description)/meshes/chassis.stl" scale="0.001 0.001 0.001"/>
+                    <mesh filename="package://omniseer_description/meshes/chassis.stl" scale="0.001 0.001 0.001"/>
                 </xacro:unless>
             </geometry>
@@ -151,5 +151,5 @@
                 </xacro:if>
                 <xacro:unless value="${use_ci_geometry}">
-                    <mesh filename="file://$(find omniseer_description)/meshes/lidar_top.stl" scale="0.001 0.001 0.001"/>
+                    <mesh filename="package://omniseer_description/meshes/lidar_top.stl" scale="0.001 0.001 0.001"/>
                 </xacro:unless>
             </geometry>
@@ -164,5 +164,5 @@
                 </xacro:if>
                 <xacro:unless value="${use_ci_geometry}">
-                    <mesh filename="file://$(find omniseer_description)/meshes/lidar_top.stl" scale="0.001 0.001 0.001"/>
+                    <mesh filename="package://omniseer_description/meshes/lidar_top.stl" scale="0.001 0.001 0.001"/>
                 </xacro:unless>
             </geometry>

Commit message: fix(sim): clean up detector scene visuals

File: ros_ws/src/omniseer_description/urdf/xacro/omniseer.urdf.xacro (robot description, xacro)
@@ -16,4 +16,5 @@
     <xacro:property name="wheel_radius" value="0.0485"/>
     <xacro:property name="wheel_width" value="0.0445"/>
+    <xacro:property name="lidar_top_mesh_origin_z" value="-0.15209671"/>
     <!-- Links -->
     <link name="fl_wheel">
@@ -145,12 +146,8 @@
             <inertia ixx="0.0002051785615782703" iyy="0.0002051785615782599" izz="0.000370076669349746" ixy="9.281393431592715e-18" iyz="4.224665266698078e-18" ixz="1.2566166227386013e-18" />
         </inertial>
+        <xacro:if value="${use_ci_geometry}">
         <visual name="lidar_top_visual">
             <geometry>
-                <xacro:if value="${use_ci_geometry}">
-                    <cylinder radius="0.045" length="0.03"/>
-                </xacro:if>
-                <xacro:unless value="${use_ci_geometry}">
-                    <mesh filename="package://omniseer_description/meshes/lidar_top.stl" scale="0.001 0.001 0.001"/>
-                </xacro:unless>
+                <cylinder radius="0.045" length="0.03"/>
             </geometry>
             <material name='sensor_mat'>
@@ -158,14 +155,31 @@
             </material>
         </visual>
+        </xacro:if>
+        <xacro:unless value="${use_ci_geometry}">
+        <visual name="lidar_top_visual">
+            <origin xyz="0.0 0.0 ${lidar_top_mesh_origin_z}" rpy="0.0 -0.0 0.0" />
+            <geometry>
+                <mesh filename="package://omniseer_description/meshes/lidar_top.stl" scale="0.001 0.001 0.001"/>
+            </geometry>
+            <material name='sensor_mat'>
+                <color rgba="${sensor_rgba}"/>
+            </material>
+        </visual>
+        </xacro:unless>
+        <xacro:if value="${use_ci_geometry}">
         <collision name="lidar_top_collision">
             <geometry>
-                <xacro:if value="${use_ci_geometry}">
-                    <cylinder radius="0.045" length="0.03"/>
-                </xacro:if>
-                <xacro:unless value="${use_ci_geometry}">
-                    <mesh filename="package://omniseer_description/meshes/lidar_top.stl" scale="0.001 0.001 0.001"/>
-                </xacro:unless>
-            </geometry>
-        </collision>
+                <cylinder radius="0.045" length="0.03"/>
+            </geometry>
+        </collision>
+        </xacro:if>
+        <xacro:unless value="${use_ci_geometry}">
+        <collision name="lidar_top_collision">
+            <origin xyz="0.0 0.0 ${lidar_top_mesh_origin_z}" rpy="0.0 -0.0 0.0" />
+            <geometry>
+                <mesh filename="package://omniseer_description/meshes/lidar_top.stl" scale="0.001 0.001 0.001"/>
+            </geometry>
+        </collision>
+        </xacro:unless>
     </link>
     <link name="sonar_link">

Commit message: feat(bringup): tune sim autonomy vision load

File: ros_ws/src/omniseer_description/urdf/xacro/omniseer.urdf.xacro (robot description, xacro)
@@ -2,5 +2,11 @@
 <robot xmlns:xacro="http://www.ros.org/wiki/xacro" name="omniseer" xmlns:gz="http://gazebosim.org/schema">
     <xacro:arg name="use_ci_geometry" default="false"/>
+    <xacro:arg name="sim_camera_width" default="1920"/>
+    <xacro:arg name="sim_camera_height" default="1080"/>
+    <xacro:arg name="sim_camera_update_rate" default="30"/>
     <xacro:property name="use_ci_geometry" value="$(arg use_ci_geometry)"/>
+    <xacro:property name="sim_camera_width" value="$(arg sim_camera_width)"/>
+    <xacro:property name="sim_camera_height" value="$(arg sim_camera_height)"/>
+    <xacro:property name="sim_camera_update_rate" value="$(arg sim_camera_update_rate)"/>
     <xacro:property name="min_vel" value="-50"/>
     <xacro:property name="max_vel" value="50"/>
@@ -335,5 +341,5 @@
     <gazebo reference="camera_link">
         <sensor name="front_camera" type="camera">
-            <update_rate>30</update_rate>
+            <update_rate>${sim_camera_update_rate}</update_rate>
             <always_on>1</always_on>
             <topic>front_camera/image</topic>
@@ -341,6 +347,6 @@
                 <horizontal_fov>1.309</horizontal_fov>
                 <image>
-                    <width>1920</width>
-                    <height>1080</height>
+                    <width>${sim_camera_width}</width>
+                    <height>${sim_camera_height}</height>
                     <format>R8G8B8</format>
                 </image>
